File: pcb/Legoduino.brd (EAGLE design)
At the start: 80 x 80 mm, 91 parts, among them CON11 ISP-AVR, CON2 PIN(1+16)X3_DS, IC1 NCP3170ADR2G, IC2 RN-42, IC3 MIC5205-5.0YM5, IC4 ATMEGA2560-16AU, IC5 UG-2864HSWEG01_SPI, IC6 MIC5205-3.6YM5, IC7 MIC5205-3.3YM5, IC8 BD6221F-E2, IC9 BD6221F-E2, SW4 RST, Y1 CSTCE16M0V53-R0 16MHZ

Commit message: .
Parts:
- removed C27: 470p, PN_default:0603
- removed C28: 2u2, PN_default:0603
- removed C29: 1u, PN_default:0603
- removed IC7: MIC5205-3.3YM5, PN_IC:SOT23-5
- removed Y1: CSTCE16M0V53-R0 16MHZ, SmartPrj:RESONATOR
- added CON5, CON6: (no value), pins:PIN2X1C
- added T2, T3: IRLML2502, PN_mosfet:SOT23
- added X1: AWSCR-16.00CV-T, PN_quartz:CERAMIC_3.7X3.1
- C11, C12, C2, C8: value 22u -> 22u/16V; device PN_default:1206 -> PN_default:1210
- C13: value 470p -> 22u/10V; device PN_default:0603 -> Pietrucha:SMC_A
- C22: value 2u2 -> 22u/10V; device PN_default:0603 -> Pietrucha:SMC_A
- C23: value 1u -> 22u/16V; device PN_default:0603 -> PN_default:1210
- C24: value 470p -> 22u/16V; device PN_default:0603 -> PN_default:1210
- CON3, CON4: device pins:PIN2X1B -> pins:PIN2X1C
- IC3: value MIC5205-5.0YM5 -> LF33CDT; device PN_IC:SOT23-5 -> PN_LDO:DPAK
- IC6: value MIC5205-3.6YM5 -> TLV70235DBV; device PN_IC:SOT23-5 -> PN_LDO:SOT23-5
- R25: value N.C. -> 100R
- R26: value 10k -> 100R
- T1: value (none) -> IRLML2502; device PN_default:SOT23 -> PN_mosfet:SOT23
- moved R26 107.4 mm to (-33.0, -40.6), turned to 0 degrees
- moved C23 97.0 mm to (-38.4, -22.9), turned to 0 degrees
- moved T1 96.6 mm to (-38.4, -29.0)
- moved R25 96.4 mm to (-33.5, -19.1)
- moved C24 85.2 mm to (-38.4, -35.6), turned to 0 degrees
- moved C13 70.3 mm to (-17.0, -9.65), turned to 0 degrees
- moved C22 67.9 mm to (-17.0, -14.5), turned to 0 degrees
- moved IC3 65.3 mm to (-14.5, -2.29), turned to 0 degrees
- moved IC6 41.0 mm to (-6.86, -4.06), turned to 0 degrees
- moved CON11 26.2 mm to (39.4, 68.8)
- moved IC2 22.8 mm to (17.0, 44.3), turned to 270 degrees
- moved Y2 7.98 mm to (15.2, 64.8)
- moved C20 6.10 mm to (61.0, 40.1)
- moved C1 5.34 mm to (25.7, 70.4)
- moved C7 5.34 mm to (33.3, 68.1)
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Connections:
- removed net +5VP: C10.1, C11.1, C15.+, C2.1, C26.2, IC6.1, IC6.3, L1.2, POWER.2, POWER.5, R12.2, R25.2, R27.1, Y2.+
- removed net N$28 (its old number): C24.2, IC6.4
- new net N$26: CON5.1, T3.3
- net +3V3: now also C13.+, IC3.3; no longer C28.2, IC7.5
- net +5V: now also C10.1, C11.1, C15.+, C2.1, C22.+, C26.2, IC3.1, IC6.1, IC6.3, L1.2, POWER.2, POWER.5, R12.2, R27.1, Y2.+; no longer C22.2, C29.2, IC3.5, IC7.1, IC7.3, R25.1
- net 42: now also T2.1; no longer R26.1
- net GND: now also C13.-, C22.-, C23.2, C24.2, T2.2, T3.2, X1.0; no longer C13.1, C22.1, C23.1, C24.1, C27.1, C28.1, C29.1, IC7.2, Y1.2
- net N$24: now also R25.2, T3.1; no longer C13.2, IC3.4
- net N$25: now also T2.3; no longer T1.3
- net N$31: now also CON6.1, T1.3; no longer C27.2, IC7.4
- net OC_PWM1: now also R25.1
- net OC_PWM2: now also R26.1
- net VIN: now also C23.1, C24.1, CON5.2, CON6.2; no longer C23.2, IC3.1, IC3.3
- net XTAL1: now also X1.2; no longer Y1.3
- net XTAL2: now also X1.1; no longer Y1.1
Routing:
- removed copper zone on layer 1, net +5VP
Other:
- board text removed: "P-|>|-N"
