File: pcb/Legoduino.sch (EAGLE design)
At the start: 91 parts, among them CON11 ISP-AVR, CON2 PIN(1+16)X3_DS, IC1 NCP3170ADR2G, IC2 RN-42, IC3 MIC5205-5.0YM5, IC4 ATMEGA2560-16AU, IC5 UG-2864HSWEG01_SPI, IC6 MIC5205-3.6YM5, IC7 MIC5205-3.3YM5, IC8 BD6221F-E2, IC9 BD6221F-E2, SW4 RST, Y1 CSTCE16M0V53-R0 16MHZ

Commit message: .
Parts:
- removed C27: 470p, PN_default:C0603
- removed C28: 2u2, PN_default:C0603
- removed C29: 1u, PN_default:C0603
- removed IC7: MIC5205-3.3YM5, PN_IC:MIC5205-3.3YM5
- removed Y1: CSTCE16M0V53-R0 16MHZ, SmartPrj:RESONATORMU
- added CON5, CON6: (no value), pins:PIN2X1C
- added T2, T3: IRLML2502, PN_mosfet:IRLML2502
- added X1: AWSCR-16.00CV-T, PN_quartz:AWSCR-16.00CV-T
- C11, C12, C2, C8: value 22u -> 22u/16V; device PN_default:C1206 -> PN_default:C1210
- C13: value 470p -> 22u/10V; device PN_default:C0603 -> Pietrucha:CE-SMC_A
- C22: value 2u2 -> 22u/10V; device PN_default:C0603 -> Pietrucha:CE-SMC_A
- C23: value 1u -> 22u/16V; device PN_default:C0603 -> PN_default:C1210
- C24: value 470p -> 22u/16V; device PN_default:C0603 -> PN_default:C1210
- CON3, CON4: device pins:PIN2X1B -> pins:PIN2X1C
- IC3: value MIC5205-5.0YM5 -> LF33CDT; device PN_IC:MIC5205-5.0YM5 -> PN_LDO:LF33CDT
- IC6: value MIC5205-3.6YM5 -> TLV70235DBV; device PN_IC:MIC5205-3.6YM5 -> PN_LDO:TLV70235DBV
- R25: value N.C. -> 100R
- R26: value 10k -> 100R
- T1: value (none) -> IRLML2502; device PN_default:NPN-SOT23 -> PN_mosfet:IRLML2502
Connections:
- removed net +5VP: C10.1, C11.1, C15.+, C2.1, C26.2, IC6.EN, IC6.IN, L1.2, POWER.2, POWER.5, R12.2, R25.2, R27.1, Y2.+
- net +3V3: now also C13.+, IC3.OUT; no longer C28.2, IC7.OUT
- net +5V: now also C10.1, C11.1, C15.+, C2.1, C22.+, C26.2, IC3.IN, IC6.EN, IC6.IN, L1.2, POWER.2, POWER.5, R12.2, R27.1, Y2.+; no longer C22.2, C29.2, IC3.OUT, IC7.EN, IC7.IN, R25.1
- net 42: now also T2.G; no longer R26.1
- net GND: now also C13.-, C22.-, C23.2, C24.2, T1.S, T2.S, T3.S, X1.0; no longer C13.1, C22.1, C23.1, C24.1, C27.1, C28.1, C29.1, IC7.GND, T1.E, Y1.2
- net N$24: now also R25.2, T3.G; no longer C13.2, IC3.BYP
- net N$25: now also T2.D; no longer T1.C
- net N$26: now also CON5.1, T3.D; no longer R26.2, T1.B
- net N$28: now also R26.2, T1.G; no longer C24.2, IC6.BYP
- net N$31: now also CON6.1, T1.D; no longer C27.2, IC7.BYP
- net OC_PWM1: now also R25.1
- net OC_PWM2: now also R26.1
- net VIN: now also C23.1, C24.1, CON5.2, CON6.2; no longer C23.2, IC3.EN, IC3.IN
- net XTAL1: now also X1.2; no longer Y1.3
- net XTAL2: now also X1.1; no longer Y1.1
Other:
- note added: "30mA max."
- moved on the sheet: C23, C24, C25, R25, R26
